File: eagle/Power System/motor driver.sch (EAGLE design)
At the start: 15 parts

Commit message: PCB layout beta
Parts:
- removed R4, R6: 510, resistor:R-US_0207/10
- removed R5: 330, resistor:R-US_0207/10
- removed SV1: JSN-SR04 FRONT, con-lstb:MA04-1
- removed SV12: (no value), con-lsta:FE12-1
- removed SV2: JSN-SR04 LEFT, con-lstb:MA04-1
- removed SV3: JSN-SR04 RIGHT, con-lstb:MA04-1
- removed SV4: (no value), con-lsta:FE10-1
- removed SV5: (no value), con-lstb:MA04-1
- removed SV6: (no value), con-lsta:FE05-1
- removed SV7: MSP430 - LEFT, con-lsta:FE10-2
- removed SV8: MSP430 - RIGHT, con-lsta:FE10-2
- added K1: JJM1-12V, relay:JJM1-12V
- added L1: (no value), inductor-neosid:SM-B9
- added T4: 2N2222, transistor:2N2222
- R1, R3: value 330 -> (none); device resistor:R-US_0207/10 -> resistor:R-US_0207/7
- R2: value 510 -> (none); device resistor:R-US_0207/10 -> resistor:R-US_0207/7
Connections:
- removed net +3V3: SV12.1, SV4.10
- removed net +5V: SV1.4, SV12.2, SV2.4, SV3.4, SV5.4
- removed net N$1: R1.2, SV1.2
- removed net N$10: SV6.2, SV8.9
- removed net N$11: SV6.1, SV8.11
- removed net N$12: R3.1, R4.2, SV8.17
- removed net N$13: SV12.11, SV7.16
- removed net N$14: SV4.7, SV8.8
- removed net N$15: SV5.1, SV7.13
- removed net N$17: R5.2, SV3.2
- removed net N$18: SV12.5, SV8.16
- removed net N$20: R5.1, R6.2, SV8.4
- removed net N$21: SV12.4, SV8.18
- removed net N$24: SV1.3, SV2.3, SV3.3, SV8.15
- removed net N$25: SV12.8, SV8.3
- removed net N$26: SV5.2, SV7.15
- removed net N$27: SV12.6, SV8.5
- removed net N$28: SV12.7, SV8.7
- removed net N$30: SV12.9, SV7.4
- removed net N$5: R1.1, R2.2, SV8.19
- removed net N$9: SV12.10, SV7.14
- new net N$3: R1.2, R2.2, T4.B
- new net V+: R3.1
- net GND: now also T4.E; no longer R4.1, R6.1, SV1.1, SV12.3, SV2.1, SV3.1, SV4.4, SV4.9, SV5.3, SV6.5
- net N$4: now also K11.1, T4.C; no longer SV4.8, SV8.10
- net N$6: now also K11.2, R3.2; no longer SV6.4, SV8.2
- net N$7: now also L1.1; no longer R3.2, SV2.2
- net N$8: now also K12.P, L1.2; no longer SV6.3, SV8.1
Other:
- note added: "MCU"
- note removed: "3.3V 5V GND LED_A LED_B LED_C LED_D BUZZ_E MODE_T BATT_E BATT_AN"
- note removed: "5V Trig Echo GND"
- note removed: "Accelerometer, Gyro, Magnometer"
- note removed: "GND M1P1 M1P2 M2P1 M2P2"
- note removed: "Hc 06 Bluetooth Module"
- note removed: "IMU - MPU 9250"
- note removed: "Jose A. Montes Perez Enrique J. Torres Rivera Leroy Y. Gonzalez Torres ICOM4217 - 067"
- note removed: "Main Board Passthrough"
- note removed: "Motor Drivers - H bridge"
- note removed: "Proximity sensors JSN - SR04"
- note removed: "Rx Tx GND Vcc"
- note removed: "VCC GND SCLK SDA EDA ECL AD0 INT NCS FSYNC"
- moved on the sheet: R1, R2, R3
