File: eagle/Power System/Main Board -v1.1.brd (EAGLE design)
At the start: 100 x 80 mm, 52 parts, among them IC3 LM358N, T7 2N2222

Commit message: PCB layout beta
Parts:
- removed C1: 0.47uF, rcl:C025-030X050
- removed C2, C3, C5, C6: 0.1uF, capacitor-wima:C2.5-3
- removed C4, C7: 1uF, capacitor-wima:C2.5-3
- removed D1, D2, D3, D4: HLMP6, display-hp:HLMP6
- removed D5, D6, D7, D8, D9: 1N4004, diode:DO41-10
- removed IC1, IC2: (no value), v-reg:317TS
- removed IC3: LM358N, linear:DIL08
- removed PAD1, PAD2: WIREPADSMD5-2,5, wirepad:5-2,5
- removed R10: 2.3K, rcl:0204/7
- removed R11: 614, rcl:0204/7
- removed R12: 1K, rcl:0207/7
- removed R13, R15: 200, rcl:0204/7
- removed R14: 50K, rcl:0204/7
- removed R16: 220, rcl:0204/7
- removed R17: 290, rcl:0204/7
- removed R18: 4.7K, rcl:0204/7
- removed R19: 2.41K, rcl:0204/7
- removed R7: 72, rcl:0204/7
- removed R8: 1.2K, rcl:0204/7
- removed R9: 3.7K, rcl:0204/7
- removed S1, S2: RDT1034, switch:RDT1034
- removed S4: TL32PO, switch:TL3XPO
- removed SG1: F/BC35, buzzer:F/BC35
- removed T1, T2, T3, T4, T5, T6: (no value), transistor-neu-to92:TO92-EBC
- removed T7: 2N2222, transistor-neu-to92:TO18
- added SV12: To Notification panel, con-lsta:FE12
- added SV2: JSN-SR04 LEFT, con-lstb:MA04-1
- added SV3: JSN-SR04 RIGHT, con-lstb:MA04-1
- added SV4: MPU9250, con-lsta:FE10
- added SV5: HC-06, con-lstb:MA04-1
- added SV6: Motor communication\, con-lsta:FE05-1
- added SV7: MSP430 - LEFT, con-lsta:FE10-2
- added SV8: MSP430 - RIGHT, con-lsta:FE10-2
- R1, R3, R5: value 72 -> 330; device rcl:0204/7 -> resistor:0207/10
- R2, R4, R6: value 1.2K -> 510; device rcl:0204/7 -> resistor:0207/10
- SV1: value (none) -> JSN-SR04 FRONT; device con-lsta:FE12 -> con-lstb:MA04-1
- moved R3 179.5 mm to (113.0, 78.7), turned to 180 degrees
- moved R2 170.0 mm to (113.0, 47.0)
- moved SV1 167.6 mm to (94.0, 48.3)
- moved R1 159.3 mm to (113.0, 53.3), turned to 180 degrees
- moved R6 151.6 mm to (113.0, 59.7)
- moved R5 141.1 mm to (113.0, 64.8), turned to 180 degrees
- moved R4 130.8 mm to (113.0, 72.4)
Connections:
- removed net N$16: R12.2, T5.B
- removed net N$19: C3.1, D5.A, IC1.1, R13.1, R17.2
- removed net N$2: R2.1, T1.B
- removed net N$22: R14.1, T6.B
- removed net N$23: R14.2, R16.2, T7.3
- removed net N$3: D2.K, R3.1
- removed net V+: IC3.8, R16.1, S4.3, T6.E
- removed net V-: IC3.4
- new net N$30: SV12.9, SV7.4
- net +3V3: now also SV12.1, SV4.10, SV7.19; no longer C4.1, D1.A, D2.A, D3.A, D4.A, D5.C, D6.A, IC1.2, R13.2, R9.2, SV1.1
- net +5V: now also SV1.4, SV12.2, SV2.4, SV3.4, SV5.4; no longer C7.1, D7.C, D8.A, D9.C, IC2.2, R15.2, SG1.-, SV1.2
- net GND: now also R2.1, R4.1, R6.1, SV1.1, SV12.3, SV2.1, SV3.1, SV4.4, SV4.9, SV5.3, SV6.5, SV7.18, SV8.20; no longer C1.2, C2.2, C3.2, C4.2, C5.2, C6.2, C7.2, PAD2.1, R11.1, R17.1, R19.1, SV1.3, T1.E, T2.E, T3.E, T4.E, T5.E, T7.1
- net N$1: now also SV1.2; no longer D1.K
- net N$10: now also SV6.2, SV8.9; no longer C1.1, R10.2, SV1.9
- net N$11: now also SV6.1, SV8.11; no longer R8.1, SV1.5
- net N$12: now also R3.1, R4.2, SV8.17; no longer R4.1, SV1.7
- net N$13: now also SV12.11, SV7.16; no longer R10.1, R9.1, S1.A, S2.A
- net N$14: now also SV4.7, SV8.8; no longer C2.1, C5.1, D6.C, D8.C, IC1.3, IC2.3, PAD1.1, S4.2
- net N$15: now also SV5.1, SV7.13; no longer S1.B, S2.B
- net N$17: now also R5.2, SV3.2; no longer S1.A1, S2.A1
- net N$18: now also SV12.5, SV8.16; no longer R2.2, SV1.6
- net N$20: now also R5.1, R6.2, SV8.4; no longer C6.1, D7.A, IC2.1, R11.2, R15.1
- net N$21: now also SV12.4, SV8.18; no longer D9.A, SG1.+, T5.C
- net N$24: now also SV1.3, SV2.3, SV3.3, SV8.15; no longer R12.1, SV1.8
- net N$25: now also SV12.8, SV8.3; no longer R18.1, T6.C
- net N$26: now also SV5.2, SV7.15; no longer IC3.1, IC3.2, SV1.11
- net N$27: now also SV12.6, SV8.5; no longer IC3.3, R18.2, R19.2
- net N$28: now also SV12.7, SV8.7; no longer SV1.10, T7.2
- net N$4: now also SV4.8, SV8.10; no longer R4.2, T2.B
- net N$5: now also R1.1, R2.2, SV8.19; no longer D3.K, R5.2
- net N$6: now also SV6.4, SV8.2; no longer R6.1, T3.B
- net N$7: now also R3.2, SV2.2; no longer D4.K, R7.1
- net N$8: now also SV6.3, SV8.1; no longer R8.2, T4.B
- net N$9: now also SV12.10, SV7.14; no longer R6.2, SV1.4
Routing:
- net +5V: track 0.00 -> 185.0 mm
- net +3V3: track 0.00 -> 141.8 mm
- net N$25: track 0.00 -> 100.1 mm
- net N$30: track 0.00 -> 99.0 mm
- net N$13: track 0.00 -> 95.4 mm
- net N$5: track 0.00 -> 93.9 mm
- net N$9: track 0.00 -> 92.5 mm
- net N$27: track 0.00 -> 89.6 mm
- net N$12: track 0.00 -> 89.5 mm
- net N$28: track 0.00 -> 82.4 mm
- net N$24: track 0.00 -> 81.6 mm
- net N$20: track 0.00 -> 77.4 mm
- net N$11: track 0.00 -> 43.6 mm
- net N$10: track 0.00 -> 40.0 mm
- net N$26: track 0.00 -> 38.2 mm
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- added copper zone on layer 1, net GND
- added copper zone on layer 16, net GND
Other:
- board size 100 x 80 mm -> 130.8 x 102.5 mm
- board text added: "GND ECHO TRIG 5V"
- board text added: "M2P2 M2P2 M1P2 M1P1 GND"
- board text added: "VDD GND SCL SDA EDA ECL AD0 INT NCS FSYNC"
- board text added: "VDD GND TX RX"

Commit message: updated pcb
Parts:
- added SV10: (no value), con-lsta:FE12
- added SV9: (no value), con-lsta:FE20
- added U$1, U$2, U$3: (no value), holes:3,0
- moved SV2 21.6 mm to (72.5, 77.3), turned to 90 degrees
- moved SV7 16.6 mm to (8.89, 54.6)
- moved SV5 7.62 mm to (21.6, 16.5)
- moved SV1 6.35 mm to (94.0, 41.9)
Routing:
- net +5V: track 185.0 -> 246.0 mm
- net N$7: track 19.4 -> 37.1 mm
- net N$24: track 81.6 -> 98.7 mm
- net N$26: track 38.2 -> 55.0 mm
- net N$15: track 35.7 -> 52.4 mm
- net N$9: track 92.5 -> 108.4 mm
- net N$13: track 95.4 -> 111.4 mm
- net N$30: track 99.0 -> 112.8 mm
- net +3V3: track 141.8 -> 155.4 mm
- net N$1: track 20.9 -> 24.4 mm
Other:
- board size 130.8 x 102.5 mm -> 124.4 x 102.5 mm
- board text added: "Jose A. Montes Perez Enrique J. Torres Rivera Leroy Y. Gonzalez Torres ICOM 4217"

Commit message: resized main board
Parts:
- removed SV10: (no value), con-lsta:FE12
- removed SV9: (no value), con-lsta:FE20
- added SV14: JSN-SR04 BACK, con-lstb:MA04-1
- moved R4 101.3 mm to (18.0, 37.1)
- moved U$3 97.1 mm to (10.4, 90.2)
- moved R6 94.5 mm to (19.8, 43.9)
- moved R3 90.4 mm to (32.8, 37.2), turned to 0 degrees
- moved U$1 84.2 mm to (87.6, 92.2)
- moved U$2 81.8 mm to (91.4, 10.2)
- moved R5 81.5 mm to (34.3, 43.8), turned to 0 degrees
- moved SV5 81.2 mm to (89.9, 60.5), turned to 270 degrees
- moved SV3 80.1 mm to (25.4, 22.1)
- moved SV1 69.2 mm to (25.4, 32.4), turned to 180 degrees
- moved R2 66.6 mm to (47.1, 37.2)
- moved SV6 54.2 mm to (90.6, 47.0), turned to 90 degrees
- moved R1 53.7 mm to (61.8, 37.0), turned to 0 degrees
- moved SV2 45.4 mm to (66.5, 32.4), turned to 180 degrees
- moved SV4 34.0 mm to (64.0, 55.2)
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Routing:
- net +5V: track 246.0 -> 39.0 mm
- net N$25: track 100.1 -> 0.00 mm
- net N$24: track 98.7 -> 0.00 mm
- net N$5: track 93.9 -> 0.00 mm
- net N$27: track 89.6 -> 0.00 mm
- net +3V3: track 155.4 -> 72.6 mm
- net N$28: track 82.4 -> 0.00 mm
- net N$15: track 52.4 -> 127.4 mm
- net N$20: track 77.4 -> 4.37 mm
- net N$26: track 55.0 -> 122.4 mm
- net N$11: track 43.6 -> 0.00 mm
- net N$10: track 40.0 -> 0.00 mm
- net N$12: track 89.5 -> 52.2 mm
- net N$7: track 37.1 -> 0.00 mm
- net N$14: track 34.7 -> 0.00 mm
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- removed copper zone on layer 1, net GND
- removed copper zone on layer 16, net GND
Other:
- board size 124.4 x 102.5 mm -> 100.3 x 101.5 mm

Commit message: final pcb versions
Parts:
- SV1: value JSN-SR04 FRONT -> JSN-SR04
- SV14: value JSN-SR04 BACK -> JSN-SR04
- SV2: value JSN-SR04 LEFT -> JSN-SR04
- SV3: value JSN-SR04 RIGHT -> JSN-SR04
- moved U$3 80.0 mm to (9.14, 10.2)
- moved U$1 78.8 mm to (8.84, 95.1)
- moved SV6 59.0 mm to (47.0, 7.24), turned to 0 degrees
- moved R1 44.6 mm to (17.4, 40.8)
- moved R4 32.7 mm to (49.8, 44.7)
- moved R3 16.7 mm to (49.3, 39.8)
- moved R2 15.9 mm to (33.1, 44.8)
- moved SV5 14.2 mm to (90.7, 74.7), turned to 0 degrees
- moved SV12 11.5 mm to (76.2, 89.2)
- moved SV3 5.08 mm to (30.5, 22.1)
- moved SV14 5.08 mm to (71.6, 21.8)
- moved R5 4.02 mm to (33.0, 40.0)
- moved U$2 3.20 mm to (94.6, 10.2)
- moved R6 2.84 mm to (17.3, 45.2)
Connections:
- net N$27: now also SV12.7; no longer SV12.6
- net N$28: now also SV12.6; no longer SV12.7
Routing:
- net N$24: track 0.00 -> 153.9 mm
- net +5V: track 39.0 -> 183.3 mm
- net N$6: track 0.00 -> 122.5 mm
- net N$20: track 4.37 -> 126.4 mm
- net N$8: track 0.00 -> 121.4 mm
- net N$11: track 0.00 -> 77.9 mm
- net N$5: track 0.00 -> 76.2 mm
- net N$10: track 0.00 -> 73.6 mm
- net N$25: track 0.00 -> 72.8 mm
- net N$27: track 0.00 -> 63.0 mm
- net N$28: track 0.00 -> 53.6 mm
- net N$15: track 127.4 -> 158.2 mm
- net N$26: track 122.4 -> 142.3 mm
- net N$1: track 0.00 -> 18.8 mm
- net N$7: track 0.00 -> 17.3 mm
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- added copper zone on layer 1, net GND
- added copper zone on layer 16, net GND
Other:
- board size 100.3 x 101.5 mm -> 101.6 x 100 mm
- board text added: "3.3V 5V GND LED_A LED_B LED_C LED_D BUZZ_E MODE_T BATT_E BATT_AN"
- board text added: "5V TRIG ECHO GND"
- board text added: "RX TX GND VDD"
- board text removed: "VDD GND TX RX"

Commit message: final final final eagle files
Parts:
- moved SV3 5.08 mm to (25.4, 22.1), turned to 180 degrees
- moved SV14 5.08 mm to (66.5, 21.8)
- moved U$2 2.07 mm to (92.6, 10.4)
- moved U$1 1.16 mm to (9.16, 94.0)
- turned SV1 to 0 degrees
- turned SV2 to 0 degrees
Routing:
- net N$24: track 153.9 -> 141.8 mm
- net N$17: track 21.6 -> 27.1 mm
- net +5V: track 183.3 -> 178.9 mm
- net N$3: track 0.00 -> 1.27 mm
- net N$1: track 18.8 -> 19.9 mm
- net N$7: track 17.3 -> 16.3 mm
Other:
- board size 101.6 x 100 mm -> 97.8 x 99.1 mm

Commit message: added multimeter
Connections:
- new net N$2: SV12.12, SV7.12
Changed lines of the file:
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@@
 <wire x1="67.31" y1="87.63" x2="67.31" y2="88.9" width="0.4064" layer="16"/>
+</signal>
+<signal name="N$2">
+<contactref element="SV12" pad="12"/>
+<contactref element="SV7" pad="12"/>
+<wire x1="10.287" y1="67.691" x2="90.17" y2="89.154" width="0" layer="19" extent="1-1"/>
 </signal>
 </signals>

Commit message: last push
Routing:
- net N$2: track 0.00 -> 112.4 mm
Changed lines of the file:
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@@
 <layer number="14" name="Route14" color="1" fill="6" visible="no" active="no"/>
 <layer number="15" name="Route15" color="4" fill="6" visible="no" active="no"/>
-<layer number="16" name="Bottom" color="1" fill="1" visible="yes" active="yes"/>
+<layer number="16" name="Bottom" color="1" fill="1" visible="no" active="yes"/>
 <layer number="17" name="Pads" color="2" fill="1" visible="yes" active="yes"/>
 <layer number="18" name="Vias" color="2" fill="1" visible="yes" active="yes"/>
@@
 <layer number="155" name="FabDoc3" color="7" fill="1" visible="yes" active="yes"/>
 <layer number="199" name="Contour" color="7" fill="1" visible="yes" active="yes"/>
-<layer number="200" name="200bmp" color="1" fill="10" visible="yes" active="yes"/>
+<layer number="200" name="200bmp" color="1" fill="10" visible="no" active="yes"/>
 <layer number="201" name="201bmp" color="7" fill="1" visible="yes" active="yes"/>
 <layer number="202" name="202bmp" color="7" fill="1" visible="yes" active="yes"/>
@@
 <contactref element="SV12" pad="12"/>
 <contactref element="SV7" pad="12"/>
-<wire x1="10.287" y1="67.691" x2="90.17" y2="89.154" width="0" layer="19" extent="1-1"/>
+<wire x1="10.287" y1="67.691" x2="10.287" y2="67.437" width="0.4064" layer="16"/>
+<wire x1="10.287" y1="67.437" x2="8.89" y2="66.04" width="0.4064" layer="16"/>
+<wire x1="8.89" y1="66.04" x2="6.35" y2="66.04" width="0.4064" layer="16"/>
+<wire x1="6.35" y1="66.04" x2="5.08" y2="67.31" width="0.4064" layer="16"/>
+<wire x1="5.08" y1="67.31" x2="5.08" y2="78.74" width="0.4064" layer="16"/>
+<wire x1="5.08" y1="78.74" x2="17.78" y2="91.44" width="0.4064" layer="16"/>
+<wire x1="17.78" y1="91.44" x2="55.88" y2="91.44" width="0.4064" layer="16"/>
+<wire x1="55.88" y1="91.44" x2="59.69" y2="95.25" width="0.4064" layer="16"/>
+<wire x1="59.69" y1="95.25" x2="84.074" y2="95.25" width="0.4064" layer="16"/>
+<wire x1="84.074" y1="95.25" x2="90.17" y2="89.154" width="0.4064" layer="16"/>
 </signal>
 </signals>
