File: eagle/Power System/Notification area.brd (EAGLE design)
At the start: 99.1 x 96.5 mm, 61 parts, among them IC3 LM358N, T7 2N2222

Commit message: last push
Connections:
- removed net N$28: R20.2, SV1.10
- new net N$39: IC3.1, IC3.2, SV1.10
- net N$26: now also R20.2; no longer IC3.1, IC3.2
Routing:
- net N$26: track 48.7 -> 155.4 mm
- net N$39: track 0.00 -> 80.4 mm
- net N$28: track 76.3 -> 0.00 mm
Changed lines of the file:
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@@
 <layer number="14" name="Route14" color="1" fill="6" visible="no" active="no"/>
 <layer number="15" name="Route15" color="4" fill="6" visible="no" active="no"/>
-<layer number="16" name="Bottom" color="1" fill="1" visible="yes" active="yes"/>
+<layer number="16" name="Bottom" color="1" fill="1" visible="no" active="yes"/>
 <layer number="17" name="Pads" color="2" fill="1" visible="yes" active="yes"/>
 <layer number="18" name="Vias" color="2" fill="1" visible="yes" active="yes"/>
@@
 </polygon>
 <contactref element="R22" pad="2"/>
-<wire x1="97.79" y1="57.15" x2="94.615" y2="72.7075" width="0" layer="19" extent="1-1"/>
-<wire x1="99.06" y1="46.99" x2="97.79" y2="57.15" width="0" layer="19" extent="1-1"/>
-<wire x1="68.5292" y1="83.82" x2="94.615" y2="72.7075" width="0" layer="19" extent="1-1"/>
-<wire x1="54.61" y1="73.66" x2="68.5292" y2="83.82" width="0" layer="19" extent="1-1"/>
-<wire x1="45.72" y1="73.66" x2="54.61" y2="73.66" width="0" layer="19" extent="1-1"/>
-<wire x1="31.75" y1="73.66" x2="45.72" y2="73.66" width="0" layer="19" extent="1-1"/>
-<wire x1="20.32" y1="73.66" x2="31.75" y2="73.66" width="0" layer="19" extent="1-1"/>
-<wire x1="57.15" y1="55.88" x2="54.61" y2="73.66" width="0" layer="19" extent="1-1"/>
-<wire x1="65.1764" y1="41.148" x2="63.5" y2="54.61" width="0" layer="19" extent="1-1"/>
-<wire x1="61.722" y1="26.416" x2="65.1764" y2="41.148" width="0" layer="19" extent="1-1"/>
-<wire x1="58.42" y1="8.89" x2="61.722" y2="26.416" width="0" layer="19" extent="1-1"/>
-<wire x1="63.1825" y1="8.5725" x2="58.42" y2="8.89" width="0" layer="19" extent="1-1"/>
-<wire x1="45.72" y1="8.89" x2="58.42" y2="8.89" width="0" layer="19" extent="1-1"/>
-<wire x1="41.91" y1="8.89" x2="45.72" y2="8.89" width="0" layer="19" extent="1-1"/>
-<wire x1="27.94" y1="20.32" x2="41.91" y2="8.89" width="0" layer="19" extent="1-1"/>
-<wire x1="30.48" y1="27.94" x2="27.94" y2="20.32" width="0" layer="19" extent="1-1"/>
-<wire x1="20.32" y1="25.4" x2="27.94" y2="20.32" width="0" layer="19" extent="1-1"/>
-<wire x1="17.78" y1="40.64" x2="20.32" y2="25.4" width="0" layer="19" extent="1-1"/>
-<wire x1="9.779" y1="46.355" x2="17.78" y2="40.64" width="0" layer="19" extent="1-1"/>
-<wire x1="7.239" y1="50.165" x2="9.779" y2="46.355" width="0" layer="19" extent="1-1"/>
 </signal>
 <signal name="N$2">
@@
 <wire x1="57.2516" y1="39.4716" x2="57.15" y2="39.37" width="0.4064" layer="16"/>
 </signal>
-<signal name="N$28">
-<contactref element="SV1" pad="10"/>
-<contactref element="R20" pad="2"/>
-<wire x1="38.1" y1="46.3296" x2="38.1" y2="41.91" width="0.4064" layer="1"/>
-<wire x1="38.1" y1="41.91" x2="40.64" y2="39.37" width="0.4064" layer="1"/>
-<wire x1="38.1" y1="46.3296" x2="50.1904" y2="58.42" width="0.4064" layer="1"/>
-<wire x1="50.1904" y1="58.42" x2="68.58" y2="58.42" width="0.4064" layer="1"/>
-<wire x1="68.58" y1="58.42" x2="86.36" y2="76.2" width="0.4064" layer="1"/>
-<wire x1="86.36" y1="76.2" x2="86.36" y2="82.6008" width="0.4064" layer="1"/>
-<wire x1="86.36" y1="82.6008" x2="86.3092" y2="83.82" width="0.4064" layer="1"/>
-</signal>
 <signal name="N$26">
-<contactref element="IC3" pad="1"/>
 <contactref element="SV1" pad="11"/>
-<contactref element="IC3" pad="2"/>
-<wire x1="65.1764" y1="46.228" x2="65.1764" y2="48.768" width="0.4064" layer="1"/>
 <wire x1="68.58" y1="49.9872" x2="68.58" y2="55.88" width="0.4064" layer="1"/>
 <wire x1="68.58" y1="49.9872" x2="67.3608" y2="48.768" width="0.4064" layer="1"/>
-<wire x1="67.3608" y1="48.768" x2="65.1764" y2="48.768" width="0.4064" layer="1"/>
 <wire x1="68.58" y1="55.88" x2="88.9" y2="76.2" width="0.4064" layer="1"/>
 <wire x1="88.9" y1="76.2" x2="88.9" y2="82.6008" width="0.4064" layer="1"/>
 <wire x1="88.9" y1="82.6008" x2="88.8492" y2="83.82" width="0.4064" layer="1"/>
+<contactref element="R20" pad="2"/>
+<wire x1="40.64" y1="39.37" x2="39.37" y2="39.37" width="0.4064" layer="16"/>
+<wire x1="39.37" y1="39.37" x2="35.56" y2="43.18" width="0.4064" layer="16"/>
+<wire x1="35.56" y1="43.18" x2="35.56" y2="53.34" width="0.4064" layer="16"/>
+<wire x1="35.56" y1="53.34" x2="38.1" y2="55.88" width="0.4064" layer="16"/>
+<wire x1="38.1" y1="55.88" x2="38.1" y2="88.9" width="0.4064" layer="16"/>
+<wire x1="38.1" y1="88.9" x2="40.64" y2="91.44" width="0.4064" layer="16"/>
+<wire x1="40.64" y1="91.44" x2="86.36" y2="91.44" width="0.4064" layer="16"/>
+<wire x1="86.36" y1="91.44" x2="88.9" y2="88.9" width="0.4064" layer="16"/>
+<wire x1="88.9" y1="88.9" x2="88.9" y2="83.8708" width="0.4064" layer="16"/>
+<wire x1="88.9" y1="83.8708" x2="88.8492" y2="83.82" width="0.4064" layer="16"/>
 </signal>
 <signal name="N$29">
@@
 <wire x1="93.98" y1="79.6925" x2="94.615" y2="80.3275" width="0.4064" layer="16"/>
 </signal>
+<signal name="N$39">
+<contactref element="IC3" pad="1"/>
+<contactref element="IC3" pad="2"/>
+<contactref element="SV1" pad="10"/>
+<wire x1="86.3092" y1="83.82" x2="86.3092" y2="86.4108" width="0.4064" layer="16"/>
+<wire x1="86.3092" y1="86.4108" x2="83.82" y2="88.9" width="0.4064" layer="16"/>
+<wire x1="83.82" y1="88.9" x2="60.96" y2="88.9" width="0.4064" layer="16"/>
+<wire x1="60.96" y1="88.9" x2="58.42" y2="86.36" width="0.4064" layer="16"/>
+<wire x1="58.42" y1="86.36" x2="58.42" y2="81.28" width="0.4064" layer="16"/>
+<wire x1="58.42" y1="81.28" x2="63.5" y2="76.2" width="0.4064" layer="16"/>
+<wire x1="63.5" y1="76.2" x2="63.5" y2="71.12" width="0.4064" layer="16"/>
+<wire x1="63.5" y1="71.12" x2="68.58" y2="66.04" width="0.4064" layer="16"/>
+<wire x1="68.58" y1="66.04" x2="68.58" y2="58.42" width="0.4064" layer="16"/>
+<wire x1="68.58" y1="58.42" x2="71.12" y2="55.88" width="0.4064" layer="16"/>
+<wire x1="71.12" y1="55.88" x2="71.12" y2="54.7116" width="0.4064" layer="16"/>
+<wire x1="71.12" y1="54.7116" x2="65.1764" y2="48.768" width="0.4064" layer="16"/>
+<wire x1="65.1764" y1="48.768" x2="65.1764" y2="46.228" width="0.4064" layer="16"/>
+</signal>
 </signals>
