File: eagle/Power System/Wave X Motor Drivers.sch (EAGLE design)
At the start: 22 parts, among them K1 JJM1-12V, K2 JJM1-12V, K3 JJM1-12V, K4 JJM1-12V, T1 2N2222, T2 2N2222, T3 2N2222, T4 2N2222

Commit message: last push
Parts:
- added D1, D2, D3, D4: 1N4004, diode:1N4004
- added R13, R14: 0.47, resistor:R-US_0207/7
- L1, L2: device inductor-neosid:SM-B9 -> resistor:L-USL4532P
Connections:
- new net N$17: L1.2, R13.2
- new net N$18: L2.2, R14.2
- net GND: now also K12.O, K22.O, K32.O, K42.O
- net N$1: now also D3.A, K11.1; no longer K21.1
- net N$10: now also D2.A
- net N$12: now also D2.C
- net N$13: now also L1.1; no longer L1.2
- net N$14: now also R13.1; no longer L1.1
- net N$15: now also K12.P; no longer K22.P
- net N$16: now also K22.P, R14.1; no longer K12.P, L2.2
- net N$2: now also R1.2, R2.2; no longer R4.2, R5.2
- net N$3: now also D3.C, K11.2, R3.2; no longer R1.2, R2.2, T4.B
- net N$4: now also D4.A, K21.1; no longer K11.1
- net N$5: now also R4.2, R5.2, T4.B; no longer K21.2, R6.2
- net N$6: now also D4.C, K21.2, R6.2; no longer K11.2, R3.2
- net N$7: now also D1.A
- net N$9: now also D1.C
- net V+: now also K12.S, K22.S, K32.S, K42.S
Other:
- moved on the sheet: K1, K2, K3, K4, R1, R2, R3, R4, R5, R6, T1, T4
